Commit message: Update planar3R.urdf

File: julia/odes/planar3R.urdf (robot description, URDF)
Before this commit: robot ThreeLinkPlanar, 5 links, 4 joints
Links:
- removed link base_link
- removed link endeffector
- removed link lower_link
- removed link lowest_link
- removed link upper_link
- added link Lower_left; visual cylinder length=25 radius=1
- added link Lower_right; visual cylinder length=25 radius=1
- added link MiddleBase_link; visual cylinder length=2 radius=1
- added link Shoulder; visual box size=26 1 1
- added link Spine_link; visual box size=2 2 30
- added link Upper_left_arm1; visual cylinder length=2 radius=1
- added link Upper_left_arm2; visual cylinder length=2 radius=1
- added link Upper_left_arm3; visual cylinder length=20 radius=1
- added link Upper_right_arm1; visual cylinder length=2 radius=1
- added link Upper_right_arm2; visual cylinder length=2 radius=1
- added link Upper_right_arm3; visual cylinder length=20 radius=1
Joints:
- removed joint elbow
- removed joint endjoint
- removed joint shoulder
- removed joint wrist
- added joint Elbow_Left: type revolute, parent Upper_left_arm3, child Lower_left, origin xyz=0 0 -20 rpy=0 0 0, axis 1 0 0
- added joint Elbow_Right: type revolute, parent Upper_right_arm3, child Lower_right, origin xyz=0 0 -20 rpy=0 0 0, axis 1 0 0
- added joint Scapula: type prismatic, parent Spine_link, child Shoulder, origin xyz=0 0 30 rpy=0 0 0, axis 0 0 1
- added joint Shoulder_Left_1: type revolute, parent Shoulder, child Upper_left_arm1, origin xyz=-12 0 0 rpy=0 0 0, axis 0 0 1
- added joint Shoulder_Left_2: type revolute, parent Upper_left_arm1, child Upper_left_arm2, origin xyz=0 0 -2 rpy=0 0 0, axis 1 0 0
- added joint Shoulder_Left_3: type revolute, parent Upper_left_arm2, child Upper_left_arm3, origin xyz=0 0 -2 rpy=0 0 0, axis 0 0 1
- added joint Shoulder_Right_1: type revolute, parent Shoulder, child Upper_right_arm1, origin xyz=12 0 0 rpy=0 0 0, axis 0 0 1
- added joint Shoulder_Right_2: type revolute, parent Upper_right_arm1, child Upper_right_arm2, origin xyz=0 0 -2 rpy=0 0 0, axis 1 0 0
- added joint Shoulder_Right_3: type revolute, parent Upper_right_arm2, child Upper_right_arm3, origin xyz=0 0 -2 rpy=0 0 0, axis 0 0 1
- added joint Waist: type revolute, parent MiddleBase_link, child Spine_link, origin xyz=0 0 1 rpy=0 0 0, axis 0 0 1
